Commit message: nuevo urdf

File: Ensamblaje/urdf/Ensamblaje.urdf (robot description, URDF)
Before this commit: robot Ensamblaje, 4 links, 3 joints
Links:
- link antebrazo_link: geometry collision mesh filename=package://ensamblaje/meshes/antebrazo_link.STL; visual mesh filename=package://ensamblaje/meshes/antebrazo_link.STL
- link base_link: mass 0.38379446013465 -> 0.383794460088106; geometry collision mesh filename=package://ensamblaje/meshes/base_link.STL; visual mesh filename=package://ensamblaje/meshes/base_link.STL
- link brazo_link: mass 0.464063170661603 -> 0.445149570388111; geometry collision mesh filename=package://ensamblaje/meshes/brazo_link.STL; visual mesh filename=package://ensamblaje/meshes/brazo_link.STL
- link efector_link: geometry collision mesh filename=package://ensamblaje/meshes/efector_link.STL; visual mesh filename=package://ensamblaje/meshes/efector_link.STL
Joints:
- joint antebrazo_joint: origin xyz=0.21344 -0.032152 -0.01325 rpy=0 0 2.974 -> xyz=0.214 0.0032298 -0.02445 rpy=0 0 -3.1416
- joint brazo_joint: origin xyz=0 0 0.1027 rpy=0 0 0 -> xyz=0 0 0.12215 rpy=0 0 0
- joint efector_joint: origin xyz=-0.215 0 0.05135 rpy=3.1416 0 1.6173 -> xyz=-0.215 0 0.055 rpy=3.1416 0 0.046478

Commit message: Actualización Ensamblaje

File: Ensamblaje/urdf/Ensamblaje.urdf (robot description, URDF)
Before this commit: robot ensamblaje, 4 links, 3 joints
Links:
- link antebrazo_link: mass 0.366545541087837 -> 0.37688
- link base_link: mass 0.383794460088106 -> 0.38379
- link brazo_link: mass 0.445149570388111 -> 0.44515
- link efector_link: mass 0.0259619449019234 -> 0.025072
Joints:
- joint antebrazo_joint: limit lower=0 upper=0 effort=0 velocity=0 -> lower=-1 upper=1 effort=0 velocity=3; origin xyz=0.214 0.0032298 -0.02445 rpy=0 0 -3.1416 -> xyz=0.21502 0 -0.005 rpy=0 0 0.001599
- joint brazo_joint: limit lower=0 upper=0 effort=0 velocity=0 -> lower=-1 upper=1 effort=0 velocity=3; origin xyz=0 0 0.12215 rpy=0 0 0 -> xyz=0.09 0.12 0.1077 rpy=0 0 0
- joint efector_joint: limit lower=0 upper=0 effort=0 velocity=0 -> lower=-0.07 upper=0 effort=0 velocity=2; origin xyz=-0.215 0 0.055 rpy=3.1416 0 0.046478 -> xyz=0.215 0 -0.072 rpy=3.1416 0 -0.001599

Commit message: actualizacion urdf

File: Ensamblaje/urdf/Ensamblaje.urdf (robot description, URDF)
Before this commit: robot ensamblaje, 4 links, 3 joints
Joints:
- joint antebrazo_joint: limit lower=-1 upper=1 effort=0 velocity=3 -> lower=-1.5707 upper=1.5707 effort=0 velocity=1; origin xyz=0.21502 0 -0.005 rpy=0 0 0.001599 -> xyz=0.21502 0 -0.02 rpy=0 0 0
- joint brazo_joint: limit lower=-1 upper=1 effort=0 velocity=3 -> lower=-1.5707 upper=1.5707 effort=0 velocity=1; origin xyz=0.09 0.12 0.1077 rpy=0 0 0 -> xyz=0 0 0.1077 rpy=0 0 0
- joint efector_joint: limit lower=-0.07 upper=0 effort=0 velocity=2 -> lower=0 upper=0.05 effort=0 velocity=1; origin xyz=0.215 0 -0.072 rpy=3.1416 0 -0.001599 -> xyz=0.215 0 -0.01 rpy=3.1416 0 0
