Commit message: CR10A limites

File: docs-urdf/CR10A_soldadura/urdf/CR10A_2.urdf (robot description, URDF)
Before this commit: robot CR10A_2, 7 links, 6 joints
Joints:
- joint 1_joint: limit lower=-1.15 upper=1.15 effort=0 velocity=0 -> lower=-3.14 upper=3.14 effort=0 velocity=0
- joint 6_joint: limit lower=0 upper=0 effort=0 velocity=0 -> lower=-3.14 upper=3.14 effort=0 velocity=0

Commit message: CR10A limites all

File: docs-urdf/CR10A_soldadura/urdf/CR10A_2.urdf (robot description, URDF)
Before this commit: robot CR10A_2, 7 links, 6 joints
Joints:
- joint 2_joint: limit lower=-1.15 upper=1.15 effort=0 velocity=0 -> lower=-3.14 upper=3.14 effort=0 velocity=0
- joint 3_joint: limit lower=-1.15 upper=1.15 effort=0 velocity=0 -> lower=-1.39 upper=1.39 effort=0 velocity=0
- joint 4_joint: limit lower=-1.15 upper=1.15 effort=0 velocity=0 -> lower=-3.14 upper=3.14 effort=0 velocity=0
- joint 5_joint: limit lower=-1.15 upper=1.15 effort=0 velocity=0 -> lower=-3.14 upper=3.14 effort=0 velocity=0
